File: kicad/current_version/working/working.kicad_pcb (KiCad board)
At the start: 2 copper layers, 11 parts, among them J1 h4psmra, J2 h4psmra, J3 hi16p, J4 hi16p, U1 insoic14wi2cland

Commit message: ready to order boards
Parts:
- moved R2 11.2 mm to (-2.00, -5.00)
- moved R1 10.9 mm to (-2.00, -7.00)
Routing:
- net /scl_3v3: track 0.00 -> 47.1 mm, vias 0 -> 2
- net /sda_3v3: track 0.00 -> 43.7 mm, vias 0 -> 2
- net +3V3: track 0.00 -> 42.8 mm, vias 0 -> 1
- net /address: track 0.00 -> 21.2 mm
- net /cs: track 0.00 -> 18.8 mm
- net GND: track 0.00 -> 6.48 mm, vias 0 -> 1
- added copper zone on B.Cu, net GND
- added copper zone on F.Cu, net GND
Other:
- board outline added: 40 x 25 mm
Changed lines of the file:
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@@
       (outputformat 1)
       (mirror false)
-      (drillshape 1)
+      (drillshape 0)
       (scaleselection 1)
-      (outputdirectory "")
+      (outputdirectory "outputs")
     )
   )
@@
   )
   (footprint "oomlout_oomp_part_footprints:r6o472_electronic_resistor_0603_4700_ohm" (layer "F.Cu")
-    (at 6.287 0.03)
+    (at -2 -7)
     (descr "Resistor SMD 0603 (1608 Metric), square (rectangular) end terminal, IPC_7351 nominal, (Body size source: IPC-SM-782 page 72, https://www.pcb-3d.com/wordpress/wp-content/uploads/ipc-sm-782a_amendment_1_and_2.pdf), generated with kicad-footprint-generator")
     (tags "resistor")
@@
     (property "ki_keywords" "R res resistor")
     (attr smd)
-    (fp_text reference "R1" (at 0 -1.43) (layer "F.SilkS")
+    (fp_text reference "R1" (at -3 0) (layer "F.SilkS")
         (effects (font (size 1 1) (thickness 0.15)))
     )
@@
   )
   (footprint "oomlout_oomp_part_footprints:r6o472_electronic_resistor_0603_4700_ohm" (layer "F.Cu")
-    (at 6.287 2.54)
+    (at -2 -5)
     (descr "Resistor SMD 0603 (1608 Metric), square (rectangular) end terminal, IPC_7351 nominal, (Body size source: IPC-SM-782 page 72, https://www.pcb-3d.com/wordpress/wp-content/uploads/ipc-sm-782a_amendment_1_and_2.pdf), generated with kicad-footprint-generator")
     (tags "resistor")
@@
     (property "ki_keywords" "R res resistor")
     (attr smd)
-    (fp_text reference "R2" (at 0 -1.43) (layer "F.SilkS")
+    (fp_text reference "R2" (at -3 0) (layer "F.SilkS")
         (effects (font (size 1 1) (thickness 0.15)))
     )
@@
     (pad "4" smd roundrect (at 1.5 -2 270) (size 0.6 1.55) (layers "F.Cu" "F.Paste" "F.Mask") (roundrect_rratio 0.25)
       (net 4 "/scl_3v3") (pinfunction "Pin_4") (pintype "passive"))
-    (pad "MP" smd roundrect (at -2.8 1.875 270) (size 1.2 1.8) (layers "F.Cu" "F.Paste" "F.Mask") (roundrect_rratio 0.208333))
-    (pad "MP" smd roundrect (at 2.8 1.875 270) (size 1.2 1.8) (layers "F.Cu" "F.Paste" "F.Mask") (roundrect_rratio 0.208333))
+    (pad "MP" smd roundrect (at -2.8 1.875 270) (size 1.2 1.8) (layers "F.Cu" "F.Paste" "F.Mask") (roundrect_rratio 0.2083333333))
+    (pad "MP" smd roundrect (at 2.8 1.875 270) (size 1.2 1.8) (layers "F.Cu" "F.Paste" "F.Mask") (roundrect_rratio 0.2083333333))
     (model "${KICAD6_3DMODEL_DIR}/Connector_JST.3dshapes/JST_SH_SM04B-SRSS-TB_1x04-1MP_P1.00mm_Horizontal.wrl"
       (offset (xyz 0 0 0))
@@
     (pad "4" smd roundrect (at 1.5 -2 90) (size 0.6 1.55) (layers "F.Cu" "F.Paste" "F.Mask") (roundrect_rratio 0.25)
       (net 4 "/scl_3v3") (pinfunction "Pin_4") (pintype "passive"))
-    (pad "MP" smd roundrect (at -2.8 1.875 90) (size 1.2 1.8) (layers "F.Cu" "F.Paste" "F.Mask") (roundrect_rratio 0.208333))
-    (pad "MP" smd roundrect (at 2.8 1.875 90) (size 1.2 1.8) (layers "F.Cu" "F.Paste" "F.Mask") (roundrect_rratio 0.208333))
+    (pad "MP" smd roundrect (at -2.8 1.875 90) (size 1.2 1.8) (layers "F.Cu" "F.Paste" "F.Mask") (roundrect_rratio 0.2083333333))
+    (pad "MP" smd roundrect (at 2.8 1.875 90) (size 1.2 1.8) (layers "F.Cu" "F.Paste" "F.Mask") (roundrect_rratio 0.2083333333))
     (model "${KICAD6_3DMODEL_DIR}/Connector_JST.3dshapes/JST_SH_SM04B-SRSS-TB_1x04-1MP_P1.00mm_Horizontal.wrl"
       (offset (xyz 0 0 0))
@@
     (property "ki_keywords" "mounting hole")
     (attr exclude_from_pos_files)
-    (fp_text reference "H3" (at 0 -4.2) (layer "F.SilkS")
+    (fp_text reference "H3" (at -5 -0.5) (layer "F.SilkS")
         (effects (font (size 1 1) (thickness 0.15)))
     )
@@
     (property "ki_keywords" "mounting hole")
     (attr exclude_from_pos_files)
-    (fp_text reference "H1" (at 0 -4.2) (layer "F.SilkS")
+    (fp_text reference "H1" (at 3 -2.5) (layer "F.SilkS")
         (effects (font (size 1 1) (thickness 0.15)))
     )
@@
     )
   )
+  (gr_line (start -15 -12.5) (end 15 -12.5)
+    (stroke (width 0.1) (type default)) (layer "Edge.Cuts"))
+  (gr_arc (start 15 -12.5) (mid 18.535534 -11.035534) (end 20 -7.5)
+    (stroke (width 0.1) (type default)) (layer "Edge.Cuts"))
+  (gr_arc (start 20 7.5) (mid 18.535534 11.035534) (end 15 12.5)
+    (stroke (width 0.1) (type default)) (layer "Edge.Cuts"))
+  (gr_line (start 15 12.5) (end -15 12.5)
+    (stroke (width 0.1) (type default)) (layer "Edge.Cuts"))
+  (gr_arc (start -20 -7.5) (mid -18.535534 -11.035534) (end -15 -12.5)
+    (stroke (width 0.1) (type default)) (layer "Edge.Cuts"))
+  (gr_line (start 20 -7.5) (end 20 7.5)
+    (stroke (width 0.1) (type default)) (layer "Edge.Cuts"))
+  (gr_arc (start -15 12.5) (mid -18.535534 11.035534) (end -20 7.5)
+    (stroke (width 0.1) (type default)) (layer "Edge.Cuts"))
+  (gr_line (start -20 7.5) (end -20 -7.5)
+    (stroke (width 0.1) (type default)) (layer "Edge.Cuts"))
+  (segment (start 13 1.5) (end 15 1.5) (width 0.25) (layer "F.Cu") (net 1))
+  (segment (start -13 -1.5) (end -8.96 -1.5) (width 0.25) (layer "F.Cu") (net 1))
+  (segment (start -8.96 -1.5) (end -8.65 -1.81) (width 0.25) (layer "F.Cu") (net 1))
+  (via (at 15 1.5) (size 0.8) (drill 0.4) (layers "F.Cu" "B.Cu") (net 1))
+  (segment (start -3.81 -10.16) (end -2.825 -9.175) (width 0.25) (layer "F.Cu") (net 2))
+  (segment (start -3.763249 -5) (end -2.825 -5) (width 0.25) (layer "F.Cu") (net 2))
+  (segment (start -13 -0.5) (end -8.69 -0.5) (width 0.25) (layer "F.Cu") (net 2))
+  (segment (start -8.223249 -0.54) (end -3.763249 -5) (width 0.25) (layer "F.Cu") (net 2))
+  (segment (start -2.825 -9.175) (end -2.825 -7) (width 0.25) (layer "F.Cu") (net 2))
+  (segment (start -8.69 -0.5) (end -8.65 -0.54) (width 0.25) (layer "F.Cu") (net 2))
+  (segment (start -8.65 -0.54) (end -8.223249 -0.54) (width 0.25) (layer "F.Cu") (net 2))
+  (segment (start -2.825 -7) (end -2.825 -5) (width 0.25) (layer "F.Cu") (net 2))
+  (segment (start 13 0.5) (end 15 0.5) (width 0.25) (layer "F.Cu") (net 2))
+  (via (at 15 0.5) (size 0.8) (drill 0.4) (layers "F.Cu" "B.Cu") (net 2))
+  (segment (start 15 0.5) (end 12.275 -2.225) (width 0.25) (layer "B.Cu") (net 2))
+  (segment (start 4.125 -2.225) (end -3.81 -10.16) (width 0.25) (layer "B.Cu") (net 2))
+  (segment (start 12.275 -2.225) (end 4.125 -2.225) (width 0.25) (layer "B.Cu") (net 2))
+  (segment (start -13 0.5) (end -8.88 0.5) (width 0.25) (layer "F.Cu") (net 3))
+  (segment (start -2 -6.175) (end -1.175 -7) (width 0.25) (layer "F.Cu") (net 3))
+  (segment (start -8.88 0.5) (end -8.65 0.73) (width 0.25) (layer "F.Cu") (net 3))
+  (segment (start -8.65 0.73) (end -7.337538 0.73) (width 0.25) (layer "F.Cu") (net 3))
+  (segment (start -1.27 -7.095) (end -1.27 -10.16) (width 0.25) (layer "F.Cu") (net 3))
+  (segment (start -2 -4.607538) (end -2 -6.175) (width 0.25) (layer "F.Cu") (net 3))
+  (segment (start -1.175 -7) (end -1.27 -7.095) (width 0.25) (layer "F.Cu") (net 3))
+  (segment (start -7.337538 0.73) (end -2 -4.607538) (width 0.25) (layer "F.Cu") (net 3))
+  (segment (start 10.5 -0.5) (end 13 -0.5) (width 0.25) (layer "F.Cu") (net 3))
+  (via (at -11 0.5) (size 0.8) (drill 0.4) (layers "F.Cu" "B.Cu") (net 3))
+  (via (at 10.5 -0.5) (size 0.8) (drill 0.4) (layers "F.Cu" "B.Cu") (net 3))
+  (segment (start -11 0.5) (end 9.5 0.5) (width 0.25) (layer "B.Cu") (net 3))
+  (segment (start 9.5 0.5) (end 10.5 -0.5) (width 0.25) (layer "B.Cu") (net 3))
+  (segment (start -8.65 2) (end -7.971142 2) (width 0.25) (layer "F.Cu") (net 4))
+  (segment (start -10 2) (end -8.65 2) (width 0.25) (layer "F.Cu") (net 4))
+  (segment (start -1.175 -5) (end 1.27 -7.445) (width 0.25) (layer "F.Cu") (net 4))
+  (segment (start 1.27 -7.445) (end 1.27 -10.16) (width 0.25) (layer "F.Cu") (net 4))
+  (segment (start -7.971142 2) (end -1.175 -4.796142) (width 0.25) (layer "F.Cu") (net 4))
+  (segment (start -1.175 -4.796142) (end -1.175 -5) (width 0.25) (layer "F.Cu") (net 4))
+  (segment (start -13 1.5) (end -10.5 1.5) (width 0.25) (layer "F.Cu") (net 4))
+  (segment (start -10.5 1.5) (end -10 2) (width 0.25) (layer "F.Cu") (net 4))
+  (segment (start 13 -1.5) (end 11.5 -1.5) (width 0.25) (layer "F.Cu") (net 4))
+  (via (at 11.5 -1.5) (size 0.8) (drill 0.4) (layers "F.Cu" "B.Cu") (net 4))
+  (via (at -11 1.5) (size 0.8) (drill 0.4) (layers "F.Cu" "B.Cu") (net 4))
+  (segment (start 11.5 -1.5) (end 11.5 -0.474695) (width 0.25) (layer "B.Cu") (net 4))
+  (segment (start 11.5 -0.474695) (end 9.525305 1.5) (width 0.25) (layer "B.Cu") (net 4))
+  (segment (start 9.525305 1.5) (end -11 1.5) (width 0.25) (layer "B.Cu") (net 4))
+  (segment (start 3.81 -8.763249) (end 3.81 -10.16) (width 0.25) (layer "F.Cu") (net 5))
+  (segment (start -8.65 3.27) (end -8.223249 3.27) (width 0.25) (layer "F.Cu") (net 5))
+  (segment (start -8.223249 3.27) (end 3.81 -8.763249) (width 0.25) (layer "F.Cu") (net 5))
+  (segment (start -8.65 4.54) (end -8.223249 4.54) (width 0.25) (layer "F.Cu") (net 6))
+  (segment (start 6.35 -10.033249) (end 6.35 -10.16) (width 0.25) (layer "F.Cu") (net 6))
+  (segment (start -8.223249 4.54) (end 6.35 -10.033249) (width 0.25) (layer "F.Cu") (net 6))
+  (zone (net 1) (net_name "GND") (layers "F&B.Cu") (hatch edge 0.5)
+    (connect_pads (clearance 0.25))
+    (min_thickness 0.2) (filled_areas_thickness no)
+    (fill yes (thermal_gap 0.25) (thermal_bridge_width 0.25))
+    (polygon
+      (pts
+        (xy -25 -15)
+        (xy 25 -15)
+        (xy 25 15)
+        (xy -25 15)
+      )
+    )
+  )
